File: nedoPC/kicad/nedoboard.kicad_sch (KiCad schematic)
At the start: 15 parts, among them U1 74LS174, U2 74LS257, U3 74LS00, U4 74LS32, U5 74LS02, U6 74LS573, U7 74LS32

Commit message: Update nedopc
Parts:
- added J1: DE9_Plug, symbol Connector:DE9_Plug
- added R1, R2, R3, R4, R5: R, symbol Device:R
- added U8: AY-3-8910, Package_DIP:DIP-40_W15.24mm_Socket, symbol 48128:AY-3-8910
Connections:
- net D0: now also U6.19 (Q0), U8.37 (DA0)
- net D1: now also U6.18 (Q1), U8.36 (DA1)
- net D2: now also U6.17 (Q2), U8.35 (DA2)
- net D3: now also U6.16 (Q3), U8.34 (DA3)
- net D4: now also U6.15 (Q4), U8.33 (DA4)
- net D5: now also U6.14 (Q5), U8.32 (DA5)
- net GND: now also U6.7 (D5), U6.8 (D6), U6.9 (D7), R1.2, R2.2, R3.2, R4.2, R5.2, U8.1 (GND), U8.24 (~{A9})
- net /IORQ: now also U7.1
- net /RESET: now also U8.23 (~{RESET})
- net at U5.4: now also U8.27 (BDIR)
- net at U6.1 (OE): now also U7.6
- net +5V: now reaches U6.11 (Load)
- net +5V: now also U6.20 (VCC), J1.1, U8.25 (A8), U8.28 (BC2), U8.40 (VCC)
- net D7: now reaches U6.12 (Q7)
- net D7: now also U8.30 (DA7)
- net D6: now reaches U6.13 (Q6)
- net D6: now also U8.31 (DA6)
- net at U6.2 (D0): now also J1.3, R3.1
- net at U6.3 (D1): now also J1.2, R2.1
- net at U6.4 (D2): now also J1.4, R4.1
- net at U6.5 (D3): now also J1.5, R5.1
- net at U6.6 (D4): now also J1.6, R1.1
- net CAS1: now reaches U2.12 (Zc)
- net A14`: now reaches U2.4 (Za)
- net A15`: now reaches U2.7 (Zb)
- net CAS0: now reaches U2.9 (Zd)
- net at U5.10: now also U8.29 (BC1)
- net at U7.4: now also U7.3
- net A5: now reaches U7.5
- net /RD: now reaches U7.2
- no-connect marks 0 -> 3
Other:
- moved on the sheet: U6, U7A, U7B

Commit message: Update
Parts:
- added C10, C11, C12, C13, C9: C_Polarized, Capacitor_THT:CP_Radial_D8.0mm_P3.80mm, symbol Device:C_Polarized
- added C14: C, Capacitor_THT:C_Disc_D7.0mm_W2.5mm_P5.00mm, symbol Device:C
- added J2: Jack_3.5mm_5pin, 48128:jack_5_pin_3f07_FINAL, symbol 48128:AudioJack_5_pin
- added J3: Beep_R7, Connector_Wire:SolderWire-0.75sqmm_1x01_D1.25mm_OD3.5mm, symbol Connector_Generic:Conn_01x01
- added J4: Conn_01x07, Connector_PinSocket_2.54mm:PinSocket_1x07_P2.54mm_Horizontal, symbol Connector_Generic:Conn_01x07
- added J5: Conn_01x17, Connector_PinSocket_2.54mm:PinSocket_1x18_P2.54mm_Horizontal, symbol Connector_Generic:Conn_01x18
- added R10, R11, R12, R13, R14, R6, R7, R8, R9: R, Resistor_THT:R_Axial_DIN0207_L6.3mm_D2.5mm_P7.62mm_Horizontal, symbol Device:R
- added R15, R16: 330, Resistor_THT:R_Axial_DIN0207_L6.3mm_D2.5mm_P7.62mm_Horizontal, symbol Device:R
- added U11: 74LS74, Package_DIP:DIP-14_W7.62mm_Socket, symbol 74xx:74LS74
- added U12: 74LS04, Package_DIP:DIP-14_W7.62mm_Socket, symbol 74xx:74LS04
- added Y1: 3.579545Mhz, Crystal:Crystal_HC49-U_Horizontal, symbol Device:Crystal
- C1, C2, C3, C4, C5, C6, C7, C8: footprint Capacitor_THT:C_Disc_D7.5mm_W2.5mm_P5.00mm -> Capacitor_THT:C_Disc_D7.0mm_W2.5mm_P5.00mm
- J1: footprint (none) -> Connector_Dsub:DSUB-9_Male_Horizontal_P2.77x2.84mm_EdgePinOffset4.94mm_Housed_MountingHolesOffset7.48mm
- R1, R2, R3, R4, R5: footprint (none) -> Resistor_THT:R_Axial_DIN0207_L6.3mm_D2.5mm_P7.62mm_Horizontal
Connections:
- net +5V: now also C1.1, C2.1, C3.1, C4.1, C5.1, C6.1, C7.1, C8.1, U1.16 (VCC), U2.16 (VCC), U3.14 (VCC), U4.14 (VCC), U5.14 (VCC), U7.14 (VCC), C14.1, U11.1 (~{R}), U11.14 (VCC), U11.4 (~{S}), U12.14 (VCC)
- net A1: now also J5.9 (Pin_9)
- net A14: now also J5.12 (Pin_12)
- net A14`: now also J4.5 (Pin_5)
- net A15: now also J5.13 (Pin_13)
- net A15`: now also J4.6 (Pin_6)
- net A5: now also J5.14 (Pin_14)
- net CAS0: now also J4.1 (Pin_1)
- net CAS1: now also J4.2 (Pin_2)
- net CHSCR: now also J4.4 (Pin_4)
- net D0: now also J5.1 (Pin_1)
- net D1: now also J5.2 (Pin_2)
- net D2: now also J5.3 (Pin_3)
- net D3: now also J5.4 (Pin_4)
- net D4: now also J5.5 (Pin_5)
- net D5: now also J5.6 (Pin_6)
- net D6: now also J5.7 (Pin_7)
- net D7: now also J5.8 (Pin_8)
- net GND: now also C1.2, C2.2, C3.2, C4.2, C5.2, C6.2, C7.2, C8.2, C14.2, J2.1, J4.7 (Pin_7), J5.18 (Pin_18), R10.2, R11.2, R12.2, U11.7 (GND), U12.7 (GND)
- net ROM: now also J4.3 (Pin_3)
- net /IORQ: now also J5.17 (Pin_17)
- net /M1: now also J5.10 (Pin_10)
- net /RD: now also J5.16 (Pin_16)
- net /RESET: now also J5.11 (Pin_11)
- net /WR: now also J5.15 (Pin_15)
- net at U8.22 (CLOCK): now also U11.5 (Q)
- net at U8.3 (B): now also R11.1, R6.2, R7.1
- net at U8.38 (C): now also R12.1, R14.1
- net at U8.4 (A): now also R10.1, R13.1
- new net: C13.1, R14.2, R7.2
- new net: R15.2, R16.1, U12.2, U12.3
- new net: R16.2, U11.3 (C), U12.4, Y1.2
- new net: C10.2, J2.2
- new net: C9.2, J2.5
- new net: C11.2, R8.2, R9.1
- new net: C10.1, C13.2, R9.2
- new net: C12.1, R13.2, R6.1
- new net: R15.1, U12.1, Y1.1
- new net: C11.1, J3.1 (Pin_1)
- new net: C12.2, C9.1, R8.1
- new net: U11.2 (D), U11.6 (~{Q})
- no-connect marks 3 -> 42
Other:
- moved on the sheet: C7, U3E, U4E, U5D, U5E, U6, U7C, U7D, U7E, U8
