File: 128k_expander_2/expander2.kicad_pcb (KiCad board)
At the start: 2 copper layers, 57.4 x 73.8 mm, 17 parts, among them J1 OUTPUT, J3 INPUT, U1 74LS32, U2 74LS00, U3 74LS04, U4 74LS174, U5 74LS257, U6 74LS74

Commit message: Update
Routing:
- net /ROM_A14 (D70_27): track 77.3 -> 79.4 mm, vias 2 -> 1
- net /SCR_PAGE (D23_6): track 85.2 -> 86.0 mm
Other:
- board text added: "D23_4"
- board text added: "D23_6"
- board text added: "D25_13"
- board text added: "D25_14"
- board text added: "D27_3"
- board text added: "D27_4"
- board text added: "D27_5"
- board text added: "D29_1"
- board text added: "D40_9"
- board text added: "D49_5"
- board text added: "D70_27"
